File: TinyFPGA-UP.kicad_pcb (KiCad board)
At the start: 4 copper layers, 17.8 x 35.6 mm, 59 parts, among them J1 Conn_01x14, J2 Conn_01x14, J3 USB_B_Micro, J4 Conn_02x08, J5 Conn_02x03, SW1 SW_Push, U1 iCE40-UP5K-SG48, U2 MIC5504-3.3, U3 DSC6001CI2A, U4 MIC5365-1.2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

Commit message: Add comments
Parts:
- R12, R13, R14: value 100 -> 1k
- R9: value 270 -> 1k
Changed lines of the file:
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@@
       (effects (font (size 1 1) (thickness 0.15)))
     )
-    (fp_text value 270 (at 0 1.17 90) (layer F.Fab)
+    (fp_text value 1k (at 0 1.17 90) (layer F.Fab)
       (effects (font (size 1 1) (thickness 0.15)))
     )
@@
       (effects (font (size 1 1) (thickness 0.15)))
     )
-    (fp_text value 100 (at 0 1.17 270) (layer F.Fab)
+    (fp_text value 1k (at 0 1.17 270) (layer F.Fab)
       (effects (font (size 1 1) (thickness 0.15)))
     )
@@
       (effects (font (size 1 1) (thickness 0.15)))
     )
-    (fp_text value 100 (at 0 1.17 270) (layer F.Fab)
+    (fp_text value 1k (at 0 1.17 270) (layer F.Fab)
       (effects (font (size 1 1) (thickness 0.15)))
     )
@@
       (effects (font (size 1 1) (thickness 0.15)))
     )
-    (fp_text value 100 (at 0 1.17 270) (layer F.Fab)
+    (fp_text value 1k (at 0 1.17 270) (layer F.Fab)
       (effects (font (size 1 1) (thickness 0.15)))
     )
@@
     (pad 2 smd roundrect (at 0.485 0 180) (size 0.59 0.64) (layers F.Cu F.Paste F.Mask) (roundrect_rratio 0.25)
       (net 1 GND))
-    (model ${KISYS3DMOD}/Resistor_SMD.3dshapes/R_0402_1005Metric.wrl
-      (at (xyz 0 0 0))
-      (scale (xyz 1 1 1))
-      (rotate (xyz 0 0 0))
-    )
   )
   (module Resistor_SMD:R_0402_1005Metric (layer B.Cu)
@@
   (segment (start 153.89 102.847028) (end 153.89 101.6963) (width 0.3048) (layer F.Cu) (net 1))
   (segment (start 153.636 103.101028) (end 153.89 102.847028) (width 0.3048) (layer F.Cu) (net 1))
-  (segment (start 153.5985 101.4048) (end 153.5985 100.05) (width 0.3048) (layer F.Cu) (net 1))
-  (segment (start 153.636 104.0731) (end 153.636 103.101028) (width 0.3048) (layer F.Cu) (net 1))
+  (segment (start 153.5985 101.4048) (end 153.5985 100.05) (width 0.3048) (layer F.Cu) (net 1) (status 20))
+  (segment (start 153.636 104.0731) (end 153.636 103.101028) (width 0.3048) (layer F.Cu) (net 1) (status 10))
   (via (at 156.5 97.75) (size 0.508) (drill 0.254) (layers F.Cu B.Cu) (net 1))
   (via (at 145.75 97.75) (size 0.508) (drill 0.254) (layers F.Cu B.Cu) (net 1))

Commit message: Fix Pads Mask Clearance
Other:
- rule pad_to_mask_clearance: 0.2 -> 0.0508
Changed lines of the file:
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@@
     (pad_size 1.7 1.7)
     (pad_drill 1)
-    (pad_to_mask_clearance 0.2)
+    (pad_to_mask_clearance 0.0508)
     (solder_mask_min_width 0.25)
     (aux_axis_origin 0 0)

Commit message: Simplify hand soldering
Parts:
- moved C18 1.15 mm to (146.4, 123.2)
Routing:
- net +1V2: track 30.8 -> 33.7 mm
- net GND: track 58.9 -> 60.0 mm, vias 29 -> 27
- net +3V3: track 67.2 -> 66.0 mm
Other:
- rule solder_mask_min_width: 0.25 -> 0.1016
Changed lines of the file:
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@@
-(kicad_pcb (version 20171130) (host pcbnew "(5.0.1-3-g963ef8bb5)")
+(kicad_pcb (version 20171130) (host pcbnew "(5.1.4-0-10_14)")
   (general
     (thickness 1.6)
     (drawings 87)
-    (tracks 754)
+    (tracks 758)
     (zones 0)
     (modules 59)
@@
     (zone_45_only no)
     (trace_min 0.1524)
-    (segment_width 0.2)
-    (edge_width 0.15)
     (via_size 0.508)
     (via_drill 0.254)
@@
     (uvia_min_size 0.2)
     (uvia_min_drill 0.1)
+    (edge_width 0.15)
+    (segment_width 0.2)
     (pcb_text_width 0.3)
     (pcb_text_size 1.5 1.5)
@@
     (pad_drill 1)
     (pad_to_mask_clearance 0.0508)
-    (solder_mask_min_width 0.25)
+    (solder_mask_min_width 0.1016)
     (aux_axis_origin 0 0)
     (visible_elements FFFFFFFF)
@@
     (uvia_dia 0.508)
     (uvia_drill 0.254)
-    (diff_pair_gap 0.1524)
     (diff_pair_width 0.1524)
+    (diff_pair_gap 0.1524)
     (add_net 0A)
     (add_net 13B)
@@
     (uvia_dia 0.508)
     (uvia_drill 0.254)
-    (diff_pair_gap 0.1524)
     (diff_pair_width 0.1524)
+    (diff_pair_gap 0.1524)
     (add_net +1V2)
     (add_net +3V3)
@@
   )
   (module Capacitor_SMD:C_0402_1005Metric (layer F.Cu)
-    (at 146.375 124.4 270)
+    (at 146.375 123.25 270)
     (descr "Capacitor SMD 0402 (1005 Metric), square (rectangular) end terminal, IPC_7351 nominal, (Body size source: http://www.tortai-tech.com/upload/download/2011102023233369053.pdf), generated with kicad-footprint-generator")
     (tags capacitor)
@@
   (gr_line (start 142.246 132.0891) (end 142.246 96.5291) (layer Edge.Cuts) (width 0.15))
   (via (at 149 114.4) (size 0.508) (drill 0.254) (layers F.Cu B.Cu) (net 1) (status 30))
-  (via (at 151.2 114.4) (size 0.508) (drill 0.254) (layers F.Cu B.Cu) (net 1) (status 30))
   (via (at 153.2 116.6) (size 0.508) (drill 0.254) (layers F.Cu B.Cu) (net 1) (status 30))
-  (via (at 151.2 116.6) (size 0.508) (drill 0.254) (layers F.Cu B.Cu) (net 1) (status 30))
   (via (at 149 116.6) (size 0.508) (drill 0.254) (layers F.Cu B.Cu) (net 1) (status 30))
   (segment (start 154.1225 98.1975) (end 154.57 97.75) (width 0.3048) (layer F.Cu) (net 1) (status 30))
@@
   (segment (start 149.906 130.8191) (end 146.9809 130.8191) (width 0.3048) (layer B.Cu) (net 1) (status 10))
   (segment (start 146.903999 130.896001) (end 146.65 131.15) (width 0.3048) (layer B.Cu) (net 1))
-  (via (at 149.906 115.5791) (size 0.508) (drill 0.254) (layers F.Cu B.Cu) (net 1) (status 30))
+  (via (at 151 115.5791) (size 3) (drill 2.5) (layers F.Cu B.Cu) (net 1) (status 30))
   (via (at 145.88 106.98) (size 0.508) (drill 0.254) (layers F.Cu B.Cu) (net 1))
   (segment (start 146.02 107.12) (end 145.88 106.98) (width 0.3048) (layer F.Cu) (net 1))
@@
   (segment (start 146.37 120.24) (end 146.091928 119.961928) (width 0.3048) (layer F.Cu) (net 1))
   (segment (start 146.37 120.635) (end 146.37 120.24) (width 0.3048) (layer F.Cu) (net 1) (status 10))
-  (segment (start 146.375 125.84761) (end 146.613391 126.086001) (width 0.3048) (layer F.Cu) (net 1))
-  (segment (start 146.613391 126.086001) (end 146.86739 126.34) (width 0.3048) (layer F.Cu) (net 1))
   (via (at 146.86739 126.34) (size 0.508) (drill 0.254) (layers F.Cu B.Cu) (net 1))
-  (segment (start 146.375 124.885) (end 146.375 125.84761) (width 0.3048) (layer F.Cu) (net 1) (status 10))
   (segment (start 153.89 101.6963) (end 153.5985 101.4048) (width 0.3048) (layer F.Cu) (net 1))
   (segment (start 153.89 102.847028) (end 153.89 101.6963) (width 0.3048) (layer F.Cu) (net 1))
@@
   (via (at 156.5 98.5) (size 0.508) (drill 0.254) (layers F.Cu B.Cu) (net 1))
   (via (at 145.75 98.5) (size 0.508) (drill 0.254) (layers F.Cu B.Cu) (net 1))
+  (segment (start 146.37 123.91) (end 146.375 123.915) (width 0.3048) (layer F.Cu) (net 1) (status 30))
+  (segment (start 146.375 125.84761) (end 146.375 123.735) (width 0.3048) (layer F.Cu) (net 1))
+  (segment (start 146.86739 126.34) (end 146.375 125.84761) (width 0.3048) (layer F.Cu) (net 1))
   (segment (start 154.586 106.2731) (end 154.586 107.7731) (width 0.3048) (layer F.Cu) (net 2) (status 30))
   (segment (start 154.5879 107.775) (end 154.586 107.7731) (width 0.3048) (layer F.Cu) (net 2) (status 30))
@@
   (segment (start 147.635 107.12) (end 147.74476 107.12) (width 0.3048) (layer F.Cu) (net 2) (status 30))
   (segment (start 146.38 121.615) (end 146.37 121.605) (width 0.3048) (layer F.Cu) (net 2) (status 30))
-  (segment (start 146.37 123.91) (end 146.375 123.915) (width 0.3048) (layer F.Cu) (net 2) (status 30))
-  (segment (start 146.37 121.605) (end 146.37 123.91) (width 0.3048) (layer F.Cu) (net 2) (status 30))
   (via (at 155.500011 115.117474) (size 0.508) (drill 0.254) (layers F.Cu B.Cu) (net 2) (status 30))
   (segment (start 155.267485 115.35) (end 155.500011 115.117474) (width 0.3048) (layer F.Cu) (net 2))
@@
   (segment (start 152.44139 120.397195) (end 148.208234 120.397195) (width 0.3048) (layer In2.Cu) (net 2))
   (segment (start 152.946747 120.902552) (end 152.44139 120.397195) (width 0.3048) (layer In2.Cu) (net 2))
+  (segment (start 146.37 122.76) (end 146.375 122.765) (width 0.3048) (layer F.Cu) (net 2))
+  (segment (start 146.37 121.605) (end 146.37 122.76) (width 0.3048) (layer F.Cu) (net 2))
   (segment (start 151.786 102.0881) (end 151.636 102.2381) (width 0.1524) (layer F.Cu) (net 3) (status 30))
   (segment (start 151.786 100.41) (end 151.786 102.0881) (width 0.1524) (layer F.Cu) (net 3) (status 30))
@@
   (segment (start 154.586 109.5481) (end 154.586 109.6731) (width 0.3048) (layer F.Cu) (net 39) (status 30))
   (segment (start 152.2095 109.3113) (end 152.543668 108.977132) (width 0.3048) (layer F.Cu) (net 39) (status 10))
-  (segment (start 145.9 115.2) (end 147.9 117.2) (width 0.3048) (layer B.Cu) (net 39))
-  (segment (start 155.23001 117.2) (end 155.326011 117.103999) (width 0.3048) (layer B.Cu) (net 39))
   (segment (start 154.511 116.85) (end 155.58001 116.85) (width 0.3048) (layer F.Cu) (net 39) (status 10))
-  (segment (start 147.9 117.2) (end 155.23001 117.2) (width 0.3048) (layer B.Cu) (net 39))
-  (segment (start 155.326011 117.103999) (end 155.58001 116.85) (width 0.3048) (layer B.Cu) (net 39))
   (segment (start 155.589178 116.859168) (end 155.58001 116.85) (width 0.3048) (layer F.Cu) (net 39))
   (via (at 155.58001 116.85) (size 0.508) (drill 0.254) (layers F.Cu B.Cu) (net 39))
@@
   (segment (start 155.795832 116.859168) (end 155.589178 116.859168) (width 0.3048) (layer F.Cu) (net 39))
   (segment (start 156.13 116.525) (end 155.795832 116.859168) (width 0.3048) (layer F.Cu) (net 39) (status 10))
+  (segment (start 152.5 118.5) (end 152.5 117.951458) (width 0.3048) (layer B.Cu) (net 39))
+  (segment (start 147.75 118.586742) (end 148.413258 119.25) (width 0.3048) (layer B.Cu) (net 39))
+  (segment (start 155.23001 117.2) (end 155.326011 117.103999) (width 0.3048) (layer B.Cu) (net 39))
+  (segment (start 152.5 117.951458) (end 153.251458 117.2) (width 0.3048) (layer B.Cu) (net 39))
+  (segment (start 148.413258 119.25) (end 151.75 119.25) (width 0.3048) (layer B.Cu) (net 39))
+  (segment (start 155.326011 117.103999) (end 155.58001 116.85) (width 0.3048) (layer B.Cu) (net 39))
+  (segment (start 147.75 117.05) (end 147.75 118.586742) (width 0.3048) (layer B.Cu) (net 39))
+  (segment (start 151.75 119.25) (end 152.5 118.5) (width 0.3048) (layer B.Cu) (net 39))
+  (segment (start 153.251458 117.2) (end 155.23001 117.2) (width 0.3048) (layer B.Cu) (net 39))
+  (segment (start 145.9 115.2) (end 147.75 117.05) (width 0.3048) (layer B.Cu) (net 39))
   (segment (start 157.906001 109.636065) (end 157.906001 108.809099) (width 0.1524) (layer F.Cu) (net 40) (status 20))
   (segment (start 154.511 113.031066) (end 157.906001 109.636065) (width 0.1524) (layer F.Cu) (net 40))
